File: V2.0/SillyTinySCSI.kicad_sch (KiCad schematic)
At the start: 38 parts, among them J1 DB25_Plug, U1 74LVT125, U2 74LVT245, U3 74LVT125, U4 74LVT245

Commit message: Initial version of Centronics 50 SillyTinySCSI
Parts:
- added JP1: Term 1, Connector_PinHeader_2.54mm:PinHeader_1x02_P2.54mm_Vertical, symbol Jumper:Jumper_2_Open
- added JP2: Term 2, Connector_PinHeader_2.54mm:PinHeader_1x02_P2.54mm_Vertical, symbol Jumper:Jumper_2_Bridged
- J1: value DB25_Plug -> Centronics50_Plug; footprint ZuluSCSI:DSUB-25_Male_Vertical_Small Courtyard -> Centronics:111050113L001; symbol Connector:DB25_Plug -> 111-050-113L001:111-050-113L001; Height (none) -> 12.55; Manufacturer_Name (none) -> NorComp; Manufacturer_Part_Number (none) -> 111-050-113L001; Mouser Part Number (none) -> 636-111-050-113L001; Mouser Price/Stock (none) -> https://www.mouser.co.uk/ProductDetail/NorComp/111-050-113L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
Connections:
- net +2V8: now also JP1.1 (A), JP2.1 (A); no longer C14.1, C15.1, R10.2, R11.2, R12.2, R13.2, R14.2, R21.2, R22.2, R23.2, R24.2, R25.2, R26.2, R27.2, R28.2, R29.2, R3.2, R30.2, R31.2, R8.2
- net GND: now also J1.1, J1.10, J1.11, J1.15, J1.17, J1.19, J1.2, J1.20, J1.21, J1.22, J1.23, J1.25, J1.3, J1.35, J1.36, J1.37, J1.39, J1.4, J1.40, J1.5, J1.6, J1.8, J1.MH1, J1.MH2; no longer J1.14 (P14)
- net TERMPWR_5V: now also J1.38; no longer J1.25 (P25)
- net ~{SCSI_ACK}: now also J1.44; no longer J1.5
- net ~{SCSI_ATN}: now also J1.41; no longer J1.17 (P17)
- net ~{SCSI_BSY}: now also J1.43; no longer J1.6
- net ~{SCSI_CD}: now also J1.48; no longer J1.15 (P15)
- net ~{SCSI_DB0}: now also J1.26; no longer J1.8
- net ~{SCSI_DB1}: now also J1.27; no longer J1.21 (P21)
- net ~{SCSI_DB2}: now also J1.28; no longer J1.22 (P22)
- net ~{SCSI_DB3}: now also J1.29; no longer J1.10
- net ~{SCSI_DB4}: now also J1.30; no longer J1.23 (P23)
- net ~{SCSI_DB5}: now also J1.31; no longer J1.11
- net ~{SCSI_DB6}: now also J1.32; no longer J1.12
- net ~{SCSI_DB7}: now also J1.33; no longer J1.13
- net ~{SCSI_DBP}: now also J1.34; no longer J1.20 (P20)
- net ~{SCSI_IO}: now also J1.50; no longer J1.3
- net ~{SCSI_MSG}: now also J1.46; no longer J1.2
- net ~{SCSI_REQ}: now also J1.49; no longer J1.1
- net ~{SCSI_RST}: now also J1.45; no longer J1.4
- net ~{SCSI_SEL}: now also J1.47; no longer J1.19 (P19)
- new net: C15.1, JP1.2 (B), R12.2, R24.2, R25.2, R26.2, R27.2, R28.2, R29.2, R30.2, R31.2
- new net: C14.1, JP2.2 (B), R10.2, R11.2, R13.2, R14.2, R21.2, R22.2, R23.2, R3.2, R8.2
Other:
- moved on the sheet: R12
